File: kicad/atx-psu-controller.kicad_sch (KiCad schematic)
At the start: 23 parts, among them J1 ATX_IF, J2 HOST_IF, J3 BTN_IF, J4 LED_IF, J5 ESP_IF, Q1 BS250, Q2 2N7000, Q3 2N7000, Q4 2N3904, Q5 2N3904

Commit message: fix(sch): wire schematic symbols and embed standard library definitions
- Embed standard library symbols (Device, Transistor_FET, Transistor_BJT, Connector_Generic, power) directly into lib_symbols block

- Place all 21 components into 5 clean functional blocks aligned to the 50-mil (1.27mm) grid

- Route all wires, junctions, power rails (+5VSB, GND), and signal labels with 100% netlist parity against atx-psu-controller.kicad_pcb

- Pass Electrical Rules Check (ERC) with 0 errors
Parts:
- removed C1: 22uF, Capacitor_THT:CP_Radial_D5.0mm_P2.50mm, symbol Device:C
- removed C2, C3: 100nF, Capacitor_THT:C_Disc_D5.0mm_W2.5mm_P2.54mm, symbol Device:C
- removed D1, D2, D3: 1N5819, Diode_THT:D_DO-41_SOD81_P10.16mm_Horizontal, symbol Device:D
- removed J1: ATX_IF, Connector_PinHeader_2.54mm:PinHeader_1x03_P2.54mm_Vertical, symbol Device:J
- removed J2: HOST_IF, Connector_PinHeader_2.54mm:PinHeader_1x02_P2.54mm_Vertical, symbol Device:J
- removed J3: BTN_IF, Connector_PinHeader_2.54mm:PinHeader_1x02_P2.54mm_Vertical, symbol Device:J
- removed J4: LED_IF, Connector_PinHeader_2.54mm:PinHeader_1x02_P2.54mm_Vertical, symbol Device:J
- removed J5: ESP_IF, Connector_PinHeader_2.54mm:PinHeader_1x03_P2.54mm_Vertical, symbol Device:J
- removed Q1: BS250, Package_TO_SOT_THT:TO-92_Inline, symbol Device:Q
- removed Q2, Q3: 2N7000, Package_TO_SOT_THT:TO-92_Inline, symbol Device:Q
- removed Q4, Q5: 2N3904, Package_TO_SOT_THT:TO-92_Inline, symbol Device:Q
- removed R3: 120k, Resistor_THT:R_Axial_DIN0207_L6.3mm_D2.5mm_P7.62mm_Horizontal, symbol Device:R
- removed R7: 330R, Resistor_THT:R_Axial_DIN0207_L6.3mm_D2.5mm_P7.62mm_Horizontal, symbol Device:R
- added C_byp, C_deb: 100nF, Capacitor_THT:C_Disc_D5.0mm_W2.5mm_P2.50mm, symbol Device:C
- added C_hold: 22uF, Capacitor_THT:CP_Radial_D5.0mm_P2.50mm, symbol Device:C_Polarized
- added D1, D2, D3: 1N5819, Diode_THT:D_DO-41_SOD81_P7.62mm_Horizontal, symbol Device:D_Schottky
- added J1: ATX_PSU, Connector_PinHeader_2.54mm:PinHeader_1x03_P2.54mm_Vertical, symbol Connector_Generic:Conn_01x03
- added J2: HOST_BC250, Connector_PinHeader_2.54mm:PinHeader_1x02_P2.54mm_Vertical, symbol Connector_Generic:Conn_01x02
- added J3: CHASSIS_BTN, Connector_PinHeader_2.54mm:PinHeader_1x02_P2.54mm_Vertical, symbol Connector_Generic:Conn_01x02
- added J4: PWR_LED, Connector_PinHeader_2.54mm:PinHeader_1x02_P2.54mm_Vertical, symbol Connector_Generic:Conn_01x02
- added J5: ESP_WAKE_HDR, Connector_PinHeader_2.54mm:PinHeader_1x03_P2.54mm_Vertical, symbol Connector_Generic:Conn_01x03
- added Q1: BS250, Package_TO_SOT_THT:TO-92_Inline, symbol Transistor_FET:BS250
- added Q2, Q3: 2N7000, Package_TO_SOT_THT:TO-92_Inline, symbol Transistor_FET:2N7000
- added Q4, Q5: 2N3904, Package_TO_SOT_THT:TO-92_Inline, symbol Transistor_BJT:2N3904
- added R_bleed: 120k, Resistor_THT:R_Axial_DIN0207_L6.3mm_D2.5mm_P7.62mm_Horizontal, symbol Device:R
- added R_led: 330R, Resistor_THT:R_Axial_DIN0207_L6.3mm_D2.5mm_P7.62mm_Horizontal, symbol Device:R
Connections:
- new net +5VSB: C_byp.1, J1.1 (Pin_1), J5.1 (Pin_1), Q1.3 (S), R1.1, R_led.1
- new net BTN_IN: C_deb.1, J3.1 (Pin_1), Q1.2 (G), R1.2
- new net BTN_OUT: J2.2 (Pin_2), Q3.3 (D)
- new net ESP_WAKE: J5.2 (Pin_2), R5.1
- new net GND: C_byp.2, C_deb.2, C_hold.2, J1.3 (Pin_3), J3.2 (Pin_2), J5.3 (Pin_3), Q2.1 (S), Q3.1 (S), Q4.1 (E), Q5.1 (E), R_bleed.2
- new net HOST_ON: D1.2 (A), J2.1 (Pin_1), R4.1, R6.1
- new net LED+: J4.1 (Pin_1), R_led.2
- new net LED-: J4.2 (Pin_2), Q4.3 (C)
- new net N_ESP_CLAMP: D3.2 (A), Q5.3 (C), R5.2
- new net N_Q3_G: Q3.2 (G), R2.2
- new net N_Q4_B: Q4.2 (B), R4.2
- new net N_Q5_B: Q5.2 (B), R6.2
- new net PS_ON#: J1.2 (Pin_2), Q2.3 (D)
- new net V_GATE: C_hold.1, D1.1 (K), D2.1 (K), D3.1 (K), Q2.2 (G), R_bleed.1
- new net V_PULSE: D2.2 (A), Q1.1 (D), R2.1
Other:
- note added: "1. ATX INTERFACE & CHASSIS BUTTON"
- note added: "2. HOLD-UP TIMER & PS_ON# DRIVER"
- note added: "3. HOST INTERFACE & ACPI BUTTON MIRROR"
- note added: "4. REMOTE WAKE & INHIBIT CLAMP"
- note added: "5. POWER LED DRIVER"
